File: Mixed-Signal_Demo_PCB.kicad_sch (KiCad schematic)
At the start: 0 parts

Commit message: Lesson 12: Rest of placement, some rearrangements. Added models
Parts:
- added H101, H102, H103, H104: MountingHole, MountingHole:MountingHole_3.2mm_M3, symbol Mechanical:MountingHole
Other:
- note added: "Mounting holes (M3)"
