File: Mixed-Signal_Demo_PCB.kicad_pcb (KiCad board)
At the start: 4 copper layers, 0 parts

Commit message: Lesson 12: MCU and USB rough placement
Parts:
- added C201: 100n, Capacitor_SMD:C_0402_1005Metric, F.Cu at (268.1, 104.9)
- added C202: 1u, Capacitor_SMD:C_0603_1608Metric, F.Cu at (254.1, 95.9)
- added C203: 1u, Capacitor_SMD:C_0603_1608Metric, F.Cu at (254.1, 98.5)
- added C204: 22u, Capacitor_SMD:C_0805_2012Metric, F.Cu at (258.3, 96.2)
- added C205: 22u, Capacitor_SMD:C_0805_2012Metric, F.Cu at (258.3, 99.2)
- added C206: 22u, Capacitor_SMD:C_0805_2012Metric, F.Cu at (258.3, 102.2)
- added C207: 22u, Capacitor_SMD:C_0805_2012Metric, F.Cu at (258.3, 105.2)
- added C208: 22u, Capacitor_SMD:C_0805_2012Metric, F.Cu at (258.3, 108.2)
- added C209: DNP, Capacitor_SMD:C_0402_1005Metric, F.Cu at (268.1, 106.9)
- added C301: 10u, Capacitor_SMD:C_0603_1608Metric, F.Cu at (116.8, 92.8)
- added C302: 100n, Capacitor_SMD:C_0402_1005Metric, F.Cu at (118.2, 92.8)
- added C303: 100n, Capacitor_SMD:C_0402_1005Metric, F.Cu at (127.0, 101.8)
- added C304: 100n, Capacitor_SMD:C_0402_1005Metric, F.Cu at (129.8, 93.0)
- added C305: 100n, Capacitor_SMD:C_0402_1005Metric, F.Cu at (121.2, 90.2)
- added C306: 10n, Capacitor_SMD:C_0402_1005Metric, F.Cu at (118.2, 97.2)
- added C307: 1u, Capacitor_SMD:C_0603_1608Metric, F.Cu at (116.8, 97.8)
- added C308: 1u, Capacitor_SMD:C_0603_1608Metric, F.Cu at (115.0, 97.8)
- added C309: 10p, Capacitor_SMD:C_0402_1005Metric, F.Cu at (114.6, 94.3)
- added C310: 10p, Capacitor_SMD:C_0402_1005Metric, F.Cu at (112.0, 94.2)
- added C311: 100n, Capacitor_SMD:C_0402_1005Metric, F.Cu at (140.1, 101.9)
- added C312: 100n, Capacitor_SMD:C_0402_1005Metric, F.Cu at (120.9, 84.6)
- added C313: 100n, Capacitor_SMD:C_0402_1005Metric, F.Cu at (138.4, 89.0)
- added C401: 1n, Capacitor_SMD:C_0402_1005Metric, F.Cu at (246.5, 56.1)
- added C402: 100n, Capacitor_SMD:C_0402_1005Metric, F.Cu at (246.5, 58.1)
- added C403: 100n, Capacitor_SMD:C_0402_1005Metric, F.Cu at (246.5, 60.1)
- added C404: 100n, Capacitor_SMD:C_0402_1005Metric, F.Cu at (246.5, 62.0)
- added C405: 150p, Capacitor_SMD:C_0402_1005Metric, F.Cu at (246.5, 64.0)
- added C406: 1n, Capacitor_SMD:C_0402_1005Metric, F.Cu at (246.5, 66.0)
- added C407: 150p, Capacitor_SMD:C_0402_1005Metric, F.Cu at (249.4, 56.1)
- added C408: 150p, Capacitor_SMD:C_0402_1005Metric, F.Cu at (249.4, 58.1)
- added C409: 10u, Capacitor_SMD:C_0603_1608Metric, F.Cu at (243.1, 56.4)
- added C410: 100n, Capacitor_SMD:C_0402_1005Metric, F.Cu at (249.4, 60.1)
- added C411: 100n, Capacitor_SMD:C_0402_1005Metric, F.Cu at (249.4, 62.0)
- added C412: 10u, Capacitor_SMD:C_0603_1608Metric, F.Cu at (243.1, 58.9)
- added C413: 10u, Capacitor_SMD:C_0603_1608Metric, F.Cu at (243.1, 61.4)
- added C414: 10u, Capacitor_SMD:C_0603_1608Metric, F.Cu at (243.1, 63.9)
- added C415: 10u, Capacitor_SMD:C_0603_1608Metric, F.Cu at (243.1, 66.4)
- added C416: 100n, Capacitor_SMD:C_0402_1005Metric, F.Cu at (249.4, 64.0)
- added C501: 1n, Capacitor_SMD:C_0402_1005Metric, F.Cu at (274.5, 56.1)
- added C502: 10u, Capacitor_SMD:C_0603_1608Metric, F.Cu at (272.1, 66.3)
- added C503: 100n, Capacitor_SMD:C_0402_1005Metric, F.Cu at (274.5, 58.1)
- added C504: 100n, Capacitor_SMD:C_0402_1005Metric, F.Cu at (274.5, 60.1)
- added C505: 1n, Capacitor_SMD:C_0402_1005Metric, F.Cu at (274.5, 62.0)
- added C506: 150p, Capacitor_SMD:C_0402_1005Metric, F.Cu at (274.5, 64.0)
- added C507: 1u, Capacitor_SMD:C_0603_1608Metric, F.Cu at (272.1, 68.8)
- added D201: GREEN, LED_SMD:LED_0402_1005Metric, F.Cu at (267.4, 101.7)
- added D301: LED_RGB_E6C1206RGBC3UDA, Missing_Footprints:E6C1206RGBC3UDA, F.Cu at (118.0, 84.7)
- added D302: PESD3V3L1BA,115, Diode_SMD:D_SOD-323, F.Cu at (135.4, 76.6)
- added D303: PESD3V3L1BA,115, Diode_SMD:D_SOD-323, F.Cu at (130.1, 87.4)
- added D304: PESD3V3L1BA,115, Diode_SMD:D_SOD-323, F.Cu at (128.8, 80.9)
- added D305: PESD3V3L1BA,115, Diode_SMD:D_SOD-323, F.Cu at (133.5, 87.4)
- added D306: PESD3V3L1BA,115, Diode_SMD:D_SOD-323, F.Cu at (136.9, 87.4)
- added D401: PESD3V3L1BA,115, Diode_SMD:D_SOD-323, F.Cu at (247.3, 73.0)
- added D501: PESD3V3L1BA,115, Diode_SMD:D_SOD-323, F.Cu at (272.3, 83.3)
- added FL301: CMF3216F-900-2P-T, Missing_Footprints:CMF3216F, F.Cu at (134.8, 95.2)
- added J301: USB_C_Receptacle_USB2.0_16P, Connector_USB:USB_C_Receptacle_HRO_TYPE-C-31-M-12, F.Cu at (148.3, 95.2)
- added J302: 2x5x1.27mm, Connector_PinHeader_1.27mm:PinHeader_2x05_P1.27mm_Vertical_SMD, F.Cu at (133.7, 82.0)
- added J401: DOSIN-801-0031, Connector_Coaxial:BNC_Amphenol_B6252HB-NPP3G-50_Horizontal, F.Cu at (232.7, 89.5)
- added J501: DOSIN-801-0031, Connector_Coaxial:BNC_Amphenol_B6252HB-NPP3G-50_Horizontal, F.Cu at (261.8, 89.5)
- added L201: 10n, Inductor_SMD:L_0603_1608Metric, F.Cu at (254.1, 101.0)
- added L202: 68u, Inductor_SMD:L_0603_1608Metric, F.Cu at (254.1, 103.5)
- added L301: 10n, Inductor_SMD:L_0402_1005Metric, F.Cu at (115.9, 99.9)
- added R201: 10R, Resistor_SMD:R_0603_1608Metric, F.Cu at (254.1, 106.0)
- added R202: 1k, Resistor_SMD:R_0402_1005Metric, F.Cu at (267.1, 95.7)
- added R203: 1k, Resistor_SMD:R_0402_1005Metric, F.Cu at (267.1, 97.7)
- added R204: 100k, Resistor_SMD:R_0603_1608Metric, F.Cu at (254.1, 108.5)
- added R205: 1k, Resistor_SMD:R_0402_1005Metric, F.Cu at (267.1, 99.7)
- added R206: 22k, Resistor_SMD:R_0603_1608Metric, F.Cu at (254.1, 111.0)
- added R301: 10k, Resistor_SMD:R_0402_1005Metric, F.Cu at (123.3, 88.3)
- added R302: 10k, Resistor_SMD:R_0402_1005Metric, F.Cu at (121.2, 101.9)
- added R303: 5k1, Resistor_SMD:R_0402_1005Metric, F.Cu at (140.4, 98.3)
- added R304: 5k1, Resistor_SMD:R_0402_1005Metric, F.Cu at (140.4, 92.3)
- added R305: 0R, Resistor_SMD:R_0402_1005Metric, F.Cu at (112.0, 95.5)
- added R306: 1k5, Resistor_SMD:R_0402_1005Metric, F.Cu at (131.6, 94.2)
- added R307: 10k, Resistor_SMD:R_0402_1005Metric, F.Cu at (130.1, 99.6)
- added R308: 1k, Resistor_SMD:R_0402_1005Metric, F.Cu at (119.0, 87.5)
- added R309: 49R9, Resistor_SMD:R_0402_1005Metric, F.Cu at (130.7, 89.0)
- added R310: 1k, Resistor_SMD:R_0402_1005Metric, F.Cu at (115.2, 87.5)
- added R311: 49R9, Resistor_SMD:R_0402_1005Metric, F.Cu at (127.2, 80.3)
- added R312: 49R9, Resistor_SMD:R_0402_1005Metric, F.Cu at (133.0, 89.0)
- added R313: 1k, Resistor_SMD:R_0402_1005Metric, F.Cu at (117.1, 87.5)
- added R314: 49R9, Resistor_SMD:R_0402_1005Metric, F.Cu at (136.4, 89.0)
- added R401: 2M2, Resistor_SMD:R_0603_1608Metric, F.Cu at (243.1, 68.9)
- added R402: 1k, Resistor_SMD:R_0402_1005Metric, F.Cu at (242.5, 76.2)
- added R403: 6k8, Resistor_SMD:R_0603_1608Metric, F.Cu at (243.1, 71.5)
- added R404: 22k, Resistor_SMD:R_0402_1005Metric, F.Cu at (242.5, 78.2)
- added R405: 12k, Resistor_SMD:R_0402_1005Metric, F.Cu at (242.5, 80.2)
- added R406: 1k, Resistor_SMD:R_0402_1005Metric, F.Cu at (242.5, 82.2)
- added R407: 2M2, Resistor_SMD:R_0603_1608Metric, F.Cu at (243.1, 74.0)
- added R408: 1k, Resistor_SMD:R_0402_1005Metric, F.Cu at (242.5, 84.2)
- added R409: 49R9, Resistor_SMD:R_0402_1005Metric, F.Cu at (242.5, 86.2)
- added R410: 0R, Resistor_SMD:R_0402_1005Metric, F.Cu at (242.5, 88.2)
- added R501: 6k8, Resistor_SMD:R_0603_1608Metric, F.Cu at (272.1, 71.4)
- added R502: 22k, Resistor_SMD:R_0402_1005Metric, F.Cu at (271.6, 56.1)
- added R503: 12k, Resistor_SMD:R_0402_1005Metric, F.Cu at (271.6, 58.1)
- added R504: 49R9, Resistor_SMD:R_0402_1005Metric, F.Cu at (271.6, 60.1)
- added R505: 0R, Resistor_SMD:R_0402_1005Metric, F.Cu at (271.6, 62.1)
- added R506: 10k, Resistor_SMD:R_0402_1005Metric, F.Cu at (271.6, 64.1)
- added U201: HT7533-1, Package_TO_SOT_SMD:SOT-89-3, F.Cu at (263.9, 107.0)
- added U202: MCP6001T-E/OT, Package_TO_SOT_SMD:SOT-23-5, F.Cu at (263.1, 97.1)
- added U203: TLV62569DBV, Package_TO_SOT_SMD:SOT-23-5, F.Cu at (263.1, 101.7)
- added U301: STM32F103CBTx, Package_QFP:LQFP-48_7x7mm_P0.5mm, F.Cu at (124.0, 96.0)
- added U302: USBLC6-2SC6, Package_TO_SOT_SMD:SOT-23-6, F.Cu at (139.7, 95.2)
- added U401: MCP6001T-E/OT, Package_TO_SOT_SMD:SOT-23-5, F.Cu at (246.6, 77.6)
- added U402: MCP6001T-E/OT, Package_TO_SOT_SMD:SOT-23-5, F.Cu at (246.6, 82.2)
- added U403: ADC141S626CIMM_NOPB, Package_SO:VSSOP-10_3x3mm_P0.5mm, F.Cu at (247.7, 86.8)
- added U404: REF3033A/DBZT, Package_TO_SOT_SMD:SOT-23, F.Cu at (247.5, 69.4)
- added U501: MCP6001T-E/OT, Package_TO_SOT_SMD:SOT-23-5, F.Cu at (272.7, 79.6)
- added U502: DAC7563TDGSR, Package_SO:VSSOP-10_3x3mm_P0.5mm, F.Cu at (273.9, 74.9)
- added Y301: 16MHz, Crystal:Crystal_SMD_3225-4Pin_3.2x2.5mm, F.Cu at (113.0, 91.8)

Commit message: Lesson 12: ADC and DAC
Parts:
- R401, R403, R407, R501: footprint Resistor_SMD:R_0603_1608Metric -> Resistor_SMD:R_0402_1005Metric
- moved C504 146.2 mm to (143.3, 124.5), turned to -90 degrees
- moved C407 146.1 mm to (118.7, 121.3), turned to 90 degrees
- moved C501 145.0 mm to (145.1, 121.6), turned to 180 degrees
- moved C401 141.2 mm to (122.5, 123.5)
- moved R502 140.8 mm to (146.7, 121.1), turned to -90 degrees
- moved C408 140.5 mm to (122.0, 117.2)
- moved U404 139.9 mm to (115.3, 115.2), turned to 180 degrees
- moved C505 139.7 mm to (147.2, 119.6)
- moved C503 139.4 mm to (144.3, 108.0)
- moved R504 139.2 mm to (148.8, 125.6), turned to -90 degrees
- moved C506 139.0 mm to (148.8, 123.5), turned to -90 degrees
- moved C410 138.9 mm to (119.8, 110.0), turned to -90 degrees
- moved C414 138.7 mm to (115.2, 117.8), turned to 180 degrees
- moved C416 138.7 mm to (119.8, 113.4), turned to 90 degrees
- moved R503 138.7 mm to (148.3, 121.6)
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Connections:
- net Net-(C404-Pad1) renamed /ADC/IN_RF
- net Net-(U404-IN) renamed /ADC/ADC_REF_IN
- net Net-(U502-VOUT_A) renamed /DAC/DAC_OUT_A
- net Net-(U502-VOUT_B) renamed /DAC/DAC_OUT_B

Commit message: Lesson 12: Rest of placement, some rearrangements. Added models
Parts:
- added H101: MountingHole, MountingHole:MountingHole_3.2mm_M3, F.Cu at (111.5, 143.0)
- added H102: MountingHole, MountingHole:MountingHole_3.2mm_M3, F.Cu at (161.5, 143.0)
- added H103: MountingHole, MountingHole:MountingHole_3.2mm_M3, F.Cu at (161.5, 78.0)
- added H104: MountingHole, MountingHole:MountingHole_3.2mm_M3, F.Cu at (111.5, 78.0)
- L201: footprint Inductor_SMD:L_0603_1608Metric -> Inductor_SMD:L_0402_1005Metric
- L202: footprint Inductor_SMD:L_0603_1608Metric -> Inductor_SMD:L_Coilcraft_XxL4020
- R201: footprint Resistor_SMD:R_0603_1608Metric -> Resistor_SMD:R_0805_2012Metric
- moved R203 75.7 mm to (135.4, 126.0)
- moved R202 73.9 mm to (137.8, 126.0)
- moved C201 70.9 mm to (139.3, 123.0), turned to 90 degrees
- moved U202 70.2 mm to (136.6, 123.5)
- moved U201 68.3 mm to (137.3, 117.9)
- moved C206 67.6 mm to (133.3, 123.6), turned to 90 degrees
- moved C205 67.2 mm to (133.3, 117.8), turned to 90 degrees
- moved C209 66.3 mm to (150.0, 87.7), turned to 180 degrees
- moved C204 64.2 mm to (136.3, 114.2), turned to 180 degrees
- moved C207 62.4 mm to (146.0, 83.5), turned to -90 degrees
- moved U203 62.1 mm to (149.3, 83.5), turned to 180 degrees
- moved D201 61.4 mm to (154.2, 83.6), turned to 90 degrees
- moved R206 59.6 mm to (147.0, 86.4)
- moved R205 59.3 mm to (154.3, 85.9), turned to 90 degrees
- moved R201 58.6 mm to (137.3, 111.2), turned to -90 degrees
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Connections:
- net Net-(U202-+) renamed /Power/VREF
Other:
- board outline added: 60 x 75 mm

Commit message: Lesson 13: Routing
Parts:
- R204, R206: footprint Resistor_SMD:R_0603_1608Metric -> Resistor_SMD:R_0402_1005Metric
- moved C312 46.2 mm to (91.1, 77.5), turned to 0 degrees
- moved D301 43.4 mm to (91.2, 80.3), turned to 90 degrees
- moved R308 41.6 mm to (94.0, 79.0), turned to 180 degrees
- moved R313 39.6 mm to (94.0, 81.5), turned to 180 degrees
- moved R310 37.8 mm to (94.0, 83.1), turned to 180 degrees
- moved C313 34.5 mm to (98.9, 66.7), turned to 90 degrees
- moved R314 32.0 mm to (100.0, 66.7), turned to -90 degrees
- moved D306 29.9 mm to (101.5, 67.2), turned to 90 degrees
- moved R306 26.6 mm to (124.3, 79.2)
- moved FL301 26.2 mm to (128.1, 80.1)
- moved R409 25.9 mm to (94.1, 93.8)
- moved C413 25.9 mm to (93.3, 91.9)
- moved C209 25.3 mm to (128.8, 74.0)
- moved R204 25.1 mm to (128.8, 72.8)
- moved U302 25.0 mm to (134.4, 80.1)
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Connections:
- net /Power/BUCK_5W renamed /Power/BUCK_SW
- J302 pad 10: /MCU/SWDIO_CONN -> /MCU/NRST_CONN
- J302 pad 2: GND -> /MCU/SWDIO_CONN
- J302 pad 4: unconnected-(J302-Pin_4-Pad4) -> /MCU/SWCLK_CONN
- J302 pad 6: /MCU/NRST_CONN -> /MCU/SWO_CONN
- J302 pad 8: /MCU/SWO_CONN -> unconnected-(J302-Pin_8-Pad8)
- J302 pad 9: /MCU/SWCLK_CONN -> GND
- R308 pad 1: /MCU/TIM4_CH1 -> /MCU/TIM4_CH3
- R310 pad 1: /MCU/TIM4_CH2 -> /MCU/TIM4_CH1
- R313 pad 1: /MCU/TIM4_CH3 -> /MCU/TIM4_CH2
- U301 pad 20: unconnected-(U301-PB2-Pad20) -> DAC_NCLR
- U301 pad 21: DAC_NCLR -> DAC_NLDAC
- U301 pad 22: DAC_NLDAC -> unconnected-(U301-PB11-Pad22)
Routing:
- net +3.3V: track 0.00 -> 177.4 mm, vias 0 -> 15
- net +3.3VA: track 0.00 -> 85.3 mm, vias 0 -> 5
- net +5V: track 0.00 -> 82.5 mm, vias 0 -> 4
- net GND: track 0.00 -> 50.2 mm, vias 0 -> 91
- net /MCU/TIM4_CH1: track 0.00 -> 32.3 mm, vias 0 -> 2
- net /MCU/NRST: track 0.00 -> 29.4 mm, vias 0 -> 2
- net /MCU/TIM4_CH2: track 0.00 -> 29.1 mm, vias 0 -> 2
- net /MCU/TIM4_CH3: track 0.00 -> 28.7 mm, vias 0 -> 2
- net DAC_NCLR: track 0.00 -> 27.8 mm, vias 0 -> 2
- net DAC_NLDAC: track 0.00 -> 27.6 mm, vias 0 -> 2
- net SPI2_MOSI: track 0.00 -> 27.4 mm
- net SPI1_MISO: track 0.00 -> 23.9 mm
- net VCOM: track 0.00 -> 23.8 mm
- net /MCU/SWDIO: track 0.00 -> 22.2 mm
- net SPI1_NSS: track 0.00 -> 19.9 mm, vias 0 -> 2
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- added copper zone on F.Cu, net +3.3V
- added copper zone on F.Cu, net +3.3VA
- added copper zone on F.Cu, net +5V
- added copper zone on F.Cu, net /ADC/ADC_REF_IN
- added copper zone on F.Cu, net /ADC/ADC_VREF
- added copper zone on F.Cu, net /Power/+5V_FILT
- added copper zone on F.Cu, net /Power/BUCK_SW
- added copper zone on F.Cu, net GND
- added copper zone on In1.Cu, net GND
- added copper zone on In2.Cu, net GND
- added copper zone on F.Cu, net VBUS

Commit message: Lesson 14: Finishing touches
Routing:
- net GND: vias 91 -> 298
Other:
- board text added: "1 MOhm"
- board text added: "20Hz < BW < 20kHz"
- board text added: "50 Ohm"
- board text added: "Mixed-Signal Demo Board"
- board text added: "ON"
- board text added: "RC 8/24 REV A"
- board text added: "SWD"
- board text added: "USB"
