File: adc.kicad_sch (KiCad schematic)
At the start: 0 parts

Commit message: Lesson 7: ADC, DAC, and frontends
Parts:
- added C401, C405, C408: 150p, symbol Device:C_Small
- added C402, C403, C412, C414, C415, C417: 100n, symbol Device:C_Small
- added C404, C406: 1n, symbol Device:C_Small
- added C409, C410, C411, C413, C416: 10u, symbol Device:C_Small
- added D401: PESD3V3L1BA,115, Diode_SMD:D_SOD-323, symbol Diode:SD05_SOD323
- added J401: DOSIN-801-0031, symbol Connector:Conn_Coaxial
- added R401, R407, R408: 1k, symbol Device:R_Small
- added R402, R403: 2M2, symbol Device:R_Small
- added R404: 6k8, symbol Device:R_Small
- added R405: 22k, symbol Device:R_Small
- added R406: 12k, symbol Device:R_Small
- added R409: 49R9, symbol Device:R_Small
- added R410: 0R, symbol Device:R_Small
- added U401, U402: MCP6001T-E/OT, Package_TO_SOT_SMD:SOT-23-5, symbol Amplifier_Operational:MCP6001-OT
- added U403: REF3033A/DBZT, Package_TO_SOT_SMD:SOT-23, symbol Reference_Voltage:REF3033
- added U404: ADC141S626CIMM_NOPB, Package_SO:VSSOP-10_3x3mm_P0.5mm, symbol MissingComponents:ADC141S626
Connections:
- new net: C404.1, R404.2, R405.1
- new net: C401.1, C402.1, R401.2, R402.2
- new net: C410.1, R409.2, U403.1 (IN)
- new net: C406.1, R405.2, R406.1
- new net +3.3V: C415.1, C416.1, U404.9 (VIO)
- new net +3.3VA: C403.2, C413.1, C414.1, C417.2, U401.5 (V+), U402.5 (V+), U404.10 (VA)
- new net +5V: C409.1, R409.1
- new net ADC_IN+: C408.1, R407.2, U404.2 (-IN)
- new net ADC_IN-: C408.2, R408.2, U404.3 (+IN)
- new net ADC_SCLK: R410.1, U404.8 (SCLK)
- new net ADC_VREF: C411.1, C412.1, U403.2 (OUT), U404.1 (VREF)
- new net GND: C401.2, C403.1, C404.2, C405.2, C409.2, C411.2, C412.2, C413.2, C414.2, C415.2, C416.2, C417.1, D401.1 (A1), J401.2 (Ext), R402.1, U401.2 (V-), U402.2 (V-), U403.3 (GND), U404.4 (GND), U404.5 (GND)
- new net IN: D401.2 (A2), J401.1 (In), R401.1
- new net IN_AA_BUF_IN: C405.1, R406.2, U402.3 (+)
- new net IN_AA_BUF_OUT: C406.2, R407.1, U402.1, U402.4 (-)
- new net IN_BUF: C402.2, R403.1, U401.3 (+)
- new net IN_BUF_OUT: R404.1, U401.1, U401.4 (-)
- new net SPI1_MISO: U404.7 (DOUT)
- new net SPI1_NSS: U404.6 (NCS)
- new net SPI1_SCLK: R410.2
- new net VCOM: R403.2, R408.1
Other:
- note added: "14-Bit S/H ADC"
- note added: "3rd order Butterworth anti-aliasing (low-pass filter) fc=25kHz"
- note added: "Analogue Front-End"
- note added: "BNC Connector"
- note added: "Input voltage must be in -1.65V to +1.65V range!"
- note added: "MCP6001: I/O Rail-to-Rail. Single-Supply (1.8V to 5V). High-impedance input CMOS. Low bias currents. Unity gain stable"
- note added: "Rin = 1.1M RF filter: fc=1.1MHz"
- note added: "Single-ended to 'balanced' conversion Both ADC inputs should be at same VCOM"
- note added: "Vref = 3V3 Vref filter: fc=319Hz P(R,max)=0.1W -> I(R,max)=45mA"
- note added: "[3] ADC & Analogue Front End"

Commit message: Lesson 8: Reannotation, running ERC for schematic
Parts:
- renumbered C406 to C401, C403 to C402, C417 to C403, C402 to C404, C401 to C405, C404 to C406, C405 to C407, C413 to C409, C414 to C410, C415 to C411, C416 to C412, C409 to C413, C410 to C414, C411 to C415, C412 to C416, R403 to R401, R401 to R402, R404 to R403, R405 to R404, R406 to R405, R407 to R406, R402 to R407, U404 to U403, U403 to U404
Connections:
- net GND: now also C414.2
- net SPI1_SCLK renamed SPI1_SCK

Commit message: Lesson 8: Assigned most footprints. Added missing ones
Parts:
- C401, C402, C403, C404, C405, C406, C407, C408, C409, C410, C411, C412, C413, C414, C415, C416: footprint (none) -> Capacitor_SMD:C_0402_1005Metric
- R401, R403, R407: footprint (none) -> Resistor_SMD:R_0603_1608Metric
- R402, R404, R405, R406, R408, R409, R410: footprint (none) -> Resistor_SMD:R_0402_1005Metric
Changed lines of the file:
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@@
 			)
 		)
-		(property "Footprint" ""
+		(property "Footprint" "Resistor_SMD:R_0402_1005Metric"
 			(at 219.71 63.5 0)
 			(effects
@@
 			)
 		)
-		(property "Footprint" ""
+		(property "Footprint" "Capacitor_SMD:C_0402_1005Metric"
 			(at 152.4 67.31 0)
 			(effects
@@
 			)
 		)
-		(property "Footprint" ""
+		(property "Footprint" "Capacitor_SMD:C_0402_1005Metric"
 			(at 134.62 119.38 0)
 			(effects
@@
 			)
 		)
-		(property "Footprint" ""
+		(property "Footprint" "Capacitor_SMD:C_0402_1005Metric"
 			(at 87.63 58.42 0)
 			(effects
@@
 			)
 		)
-		(property "Footprint" ""
+		(property "Footprint" "Capacitor_SMD:C_0402_1005Metric"
 			(at 114.3 50.8 0)
 			(effects
@@
 			)
 		)
-		(property "Footprint" ""
+		(property "Footprint" "Capacitor_SMD:C_0402_1005Metric"
 			(at 124.46 119.38 0)
 			(effects
@@
 			)
 		)
-		(property "Footprint" ""
+		(property "Footprint" "Capacitor_SMD:C_0402_1005Metric"
 			(at 228.6 73.66 0)
 			(effects
@@
 			)
 		)
-		(property "Footprint" ""
+		(property "Footprint" "Capacitor_SMD:C_0402_1005Metric"
 			(at 90.17 148.59 0)
 			(effects
@@
 			)
 		)
-		(property "Footprint" ""
+		(property "Footprint" "Capacitor_SMD:C_0402_1005Metric"
 			(at 35.56 143.51 0)
 			(effects
@@
 			)
 		)
-		(property "Footprint" ""
+		(property "Footprint" "Resistor_SMD:R_0603_1608Metric"
 			(at 96.52 53.34 0)
 			(effects
@@
 			)
 		)
-		(property "Footprint" ""
+		(property "Footprint" "Resistor_SMD:R_0402_1005Metric"
 			(at 137.16 139.7 0)
 			(effects
@@
 			)
 		)
-		(property "Footprint" ""
+		(property "Footprint" "Resistor_SMD:R_0402_1005Metric"
 			(at 41.91 133.35 0)
 			(effects
@@
 			)
 		)
-		(property "Footprint" ""
+		(property "Footprint" "Capacitor_SMD:C_0402_1005Metric"
 			(at 48.26 143.51 0)
 			(effects
@@
 			)
 		)
-		(property "Footprint" ""
+		(property "Footprint" "Capacitor_SMD:C_0402_1005Metric"
 			(at 187.96 53.34 0)
 			(effects
@@
 			)
 		)
-		(property "Footprint" ""
+		(property "Footprint" "Capacitor_SMD:C_0402_1005Metric"
 			(at 91.44 119.38 0)
 			(effects
@@
 			)
 		)
-		(property "Footprint" ""
+		(property "Footprint" "Resistor_SMD:R_0402_1005Metric"
 			(at 62.23 58.42 0)
 			(effects
@@
 			)
 		)
-		(property "Footprint" ""
+		(property "Footprint" "Resistor_SMD:R_0402_1005Metric"
 			(at 157.48 60.96 0)
 			(effects
@@
 			)
 		)
-		(property "Footprint" ""
+		(property "Footprint" "Resistor_SMD:R_0402_1005Metric"
 			(at 219.71 85.09 0)
 			(effects
@@
 			)
 		)
-		(property "Footprint" ""
+		(property "Footprint" "Capacitor_SMD:C_0402_1005Metric"
 			(at 81.28 119.38 0)
 			(effects
@@
 			)
 		)
-		(property "Footprint" ""
+		(property "Footprint" "Capacitor_SMD:C_0402_1005Metric"
 			(at 81.28 64.77 0)
 			(effects
@@
 			)
 		)
-		(property "Footprint" ""
+		(property "Footprint" "Capacitor_SMD:C_0402_1005Metric"
 			(at 173.99 67.31 0)
 			(effects
@@
 			)
 		)
-		(property "Footprint" ""
+		(property "Footprint" "Resistor_SMD:R_0603_1608Metric"
 			(at 71.12 64.77 0)
 			(effects
@@
 			)
 		)
-		(property "Footprint" ""
+		(property "Footprint" "Resistor_SMD:R_0402_1005Metric"
 			(at 167.64 60.96 0)
 			(effects
@@
 			)
 		)
-		(property "Footprint" ""
+		(property "Footprint" "Resistor_SMD:R_0603_1608Metric"
 			(at 147.32 60.96 0)
 			(effects
@@
 			)
 		)
-		(property "Footprint" ""
+		(property "Footprint" "Capacitor_SMD:C_0402_1005Metric"
 			(at 173.99 44.45 0)
 			(effects
@@
 			)
 		)
-		(property "Footprint" ""
+		(property "Footprint" "Capacitor_SMD:C_0402_1005Metric"
 			(at 80.01 148.59 0)
 			(effects

Commit message: Lesson 11: Adjusted capacitor footprints and set up PCB defaults
Parts:
- C409, C412, C413, C414, C415: footprint Capacitor_SMD:C_0402_1005Metric -> Capacitor_SMD:C_0603_1608Metric
- J401: footprint (none) -> Connector_Coaxial:BNC_Amphenol_B6252HB-NPP3G-50_Horizontal
Changed lines of the file:
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@@
 			)
 		)
-		(property "Footprint" ""
+		(property "Footprint" "Connector_Coaxial:BNC_Amphenol_B6252HB-NPP3G-50_Horizontal"
 			(at 38.1 58.42 0)
 			(effects
@@
 			)
 		)
-		(property "Footprint" "Capacitor_SMD:C_0402_1005Metric"
+		(property "Footprint" "Capacitor_SMD:C_0603_1608Metric"
 			(at 134.62 119.38 0)
 			(effects
@@
 			)
 		)
-		(property "Footprint" "Capacitor_SMD:C_0402_1005Metric"
+		(property "Footprint" "Capacitor_SMD:C_0603_1608Metric"
 			(at 35.56 143.51 0)
 			(effects
@@
 			)
 		)
-		(property "Footprint" "Capacitor_SMD:C_0402_1005Metric"
+		(property "Footprint" "Capacitor_SMD:C_0603_1608Metric"
 			(at 48.26 143.51 0)
 			(effects
@@
 			)
 		)
-		(property "Footprint" "Capacitor_SMD:C_0402_1005Metric"
+		(property "Footprint" "Capacitor_SMD:C_0603_1608Metric"
 			(at 81.28 119.38 0)
 			(effects
@@
 			)
 		)
-		(property "Footprint" "Capacitor_SMD:C_0402_1005Metric"
+		(property "Footprint" "Capacitor_SMD:C_0603_1608Metric"
 			(at 80.01 148.59 0)
 			(effects

Commit message: Lesson 12: ADC and DAC
Parts:
- R401, R403, R407: footprint Resistor_SMD:R_0603_1608Metric -> Resistor_SMD:R_0402_1005Metric
Connections:
- net IN_RF: now reaches C404.1, C405.1, R402.2, R407.2
- net ADC_REF_IN: now reaches C414.1, R409.2, U404.1 (IN)
Changed lines of the file:
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@@
 		)
 	)
+	(label "ADC_REF_IN"
+		(at 49.53 133.35 0)
+		(fields_autoplaced yes)
+		(effects
+			(font
+				(size 1.27 1.27)
+			)
+			(justify left bottom)
+		)
+	)
 	(label "IN_AA_BUF_IN"
 		(at 175.26 60.96 0)
@@
 		)
 	)
+	(label "IN_RF"
+		(at 72.39 58.42 0)
+		(fields_autoplaced yes)
+		(effects
+			(font
+				(size 1.27 1.27)
+			)
+			(justify left bottom)
+		)
+	)
 	(label "IN_BUF"
 		(at 104.14 58.42 0)
@@
 			)
 		)
-		(property "Footprint" "Resistor_SMD:R_0603_1608Metric"
+		(property "Footprint" "Resistor_SMD:R_0402_1005Metric"
 			(at 96.52 53.34 0)
 			(effects
@@
 			)
 		)
-		(property "Footprint" "Resistor_SMD:R_0603_1608Metric"
+		(property "Footprint" "Resistor_SMD:R_0402_1005Metric"
 			(at 71.12 64.77 0)
 			(effects
@@
 			)
 		)
-		(property "Footprint" "Resistor_SMD:R_0603_1608Metric"
+		(property "Footprint" "Resistor_SMD:R_0402_1005Metric"
 			(at 147.32 60.96 0)
 			(effects

Commit message: Lesson 13: Routing
Changed lines of the file:
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@@
 	)
 	(global_label "SPI1_MISO"
-		(shape input)
+		(shape output)
 		(at 144.78 135.89 0)
 		(fields_autoplaced yes)

Commit message: Assembly files
Parts:
- C401, C406: MPN (none) -> C1523
- C402, C403, C404, C410, C411, C416: MPN (none) -> C1525
- C405, C407, C408: MPN (none) -> C106998
- C409, C412, C413, C414, C415: MPN (none) -> C19702
- R401, R407: MPN (none) -> C274901
- R402, R406, R408: MPN (none) -> C11702
- R403: footprint Resistor_SMD:R_0402_1005Metric -> Resistor_SMD:R_0603_1608Metric; MPN (none) -> C23212
- R404: MPN (none) -> C25768
- R405: MPN (none) -> C25752
- R409: MPN (none) -> C25120
- R410: MPN (none) -> C17168
Changed lines of the file:
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@@
 			)
 		)
+		(property "MPN" "C11702"
+			(at 219.71 63.5 0)
+			(effects
+				(font
+					(size 1.27 1.27)
+				)
+				(hide yes)
+			)
+		)
 		(pin "1"
 		)
@@
 			)
 		)
+		(property "MPN" "C1523"
+			(at 152.4 67.31 0)
+			(effects
+				(font
+					(size 1.27 1.27)
+				)
+				(hide yes)
+			)
+		)
 		(pin "2"
 		)
@@
 			)
 		)
+		(property "MPN" "C19702"
+			(at 134.62 119.38 0)
+			(effects
+				(font
+					(size 1.27 1.27)
+				)
+				(hide yes)
+			)
+		)
 		(pin "2"
 		)
@@
 			)
 		)
+		(property "MPN" "C1525"
+			(at 87.63 58.42 0)
+			(effects
+				(font
+					(size 1.27 1.27)
+				)
+				(hide yes)
+			)
+		)
 		(pin "2"
 		)
@@
 			)
 		)
+		(property "MPN" "C1525"
+			(at 114.3 50.8 0)
+			(effects
+				(font
+					(size 1.27 1.27)
+				)
+				(hide yes)
+			)
+		)
 		(pin "2"
 		)
@@
 			)
 		)
+		(property "MPN" "C1525"
+			(at 124.46 119.38 0)
+			(effects
+				(font
+					(size 1.27 1.27)
+				)
+				(hide yes)
+			)
+		)
 		(pin "2"
 		)
@@
 			)
 		)
+		(property "MPN" "C106998"
+			(at 228.6 73.66 0)
+			(effects
+				(font
+					(size 1.27 1.27)
+				)
+				(hide yes)
+			)
+		)
 		(pin "2"
 		)
@@
 			)
 		)
+		(property "MPN" "C1525"
+			(at 90.17 148.59 0)
+			(effects
+				(font
+					(size 1.27 1.27)
+				)
+				(hide yes)
+			)
+		)
 		(pin "2"
 		)
@@
 			)
 		)
+		(property "MPN" "C19702"
+			(at 35.56 143.51 0)
+			(effects
+				(font
+					(size 1.27 1.27)
+				)
+				(hide yes)
+			)
+		)
 		(pin "2"
 		)
@@
 			)
 		)
+		(property "MPN" "C274901"
+			(at 96.52 53.34 0)
+			(effects
+				(font
+					(size 1.27 1.27)
+				)
+				(hide yes)
+			)
+		)
 		(pin "1"
 		)
@@
 			)
 		)
+		(property "MPN" "C17168"
+			(at 137.16 139.7 0)
+			(effects
+				(font
+					(size 1.27 1.27)
+				)
+				(hide yes)
+			)
+		)
 		(pin "1"
 		)
@@
 			)
 		)
+		(property "MPN" "C25120"
+			(at 41.91 133.35 0)
+			(effects
+				(font
+					(size 1.27 1.27)
+				)
+				(hide yes)
+			)
+		)
 		(pin "1"
 		)
@@
 			)
 		)
+		(property "MPN" "C19702"
+			(at 48.26 143.51 0)
+			(effects
+				(font
+					(size 1.27 1.27)
+				)
+				(hide yes)
+			)
+		)
 		(pin "2"
 		)
@@
 			)
 		)
+		(property "MPN" "C1525"
+			(at 187.96 53.34 0)
+			(effects
+				(font
+					(size 1.27 1.27)
+				)
+				(hide yes)
+			)
+		)
 		(pin "2"
 		)
@@
 			)
 		)
+		(property "MPN" "C1525"
+			(at 91.44 119.38 0)
+			(effects
+				(font
+					(size 1.27 1.27)
+				)
+				(hide yes)
+			)
+		)
 		(pin "2"
 		)
@@
 			)
 		)
+		(property "MPN" "C11702"
+			(at 62.23 58.42 0)
+			(effects
+				(font
+					(size 1.27 1.27)
+				)
+				(hide yes)
+			)
+		)
 		(pin "1"
 		)
@@
 			)
 		)
+		(property "MPN" "C25768"
+			(at 157.48 60.96 0)
+			(effects
+				(font
+					(size 1.27 1.27)
+				)
+				(hide yes)
+			)
+		)
 		(pin "1"
 		)
@@
 			)
 		)
+		(property "MPN" "C11702"
+			(at 219.71 85.09 0)
+			(effects
+				(font
+					(size 1.27 1.27)
+				)
+				(hide yes)
+			)
+		)
 		(pin "1"
 		)
@@
 			)
 		)
+		(property "MPN" "C19702"
+			(at 81.28 119.38 0)
+			(effects
+				(font
+					(size 1.27 1.27)
+				)
+				(hide yes)
+			)
+		)
 		(pin "2"
 		)
@@
 			)
 		)
+		(property "MPN" "C106998"
+			(at 81.28 64.77 0)
+			(effects
+				(font
+					(size 1.27 1.27)
+				)
+				(hide yes)
+			)
+		)
 		(pin "2"
 		)
@@
 			)
 		)
+		(property "MPN" "C106998"
+			(at 173.99 67.31 0)
+			(effects
+				(font
+					(size 1.27 1.27)
+				)
+				(hide yes)
+			)
+		)
 		(pin "2"
 		)
@@
 			)
 		)
+		(property "MPN" "C274901"
+			(at 71.12 64.77 0)
+			(effects
+				(font
+					(size 1.27 1.27)
+				)
+				(hide yes)
+			)
+		)
 		(pin "1"
 		)
@@
 			)
 		)
+		(property "MPN" "C25752"
+			(at 167.64 60.96 0)
+			(effects
+				(font
+					(size 1.27 1.27)
+				)
+				(hide yes)
+			)
+		)
 		(pin "1"
 		)
@@
 			)
 		)
-		(property "Footprint" "Resistor_SMD:R_0402_1005Metric"
+		(property "Footprint" "Resistor_SMD:R_0603_1608Metric"
 			(at 147.32 60.96 0)
 			(effects
@@
 			)
 		)
+		(property "MPN" "C23212"
+			(at 147.32 60.96 0)
+			(effects
+				(font
+					(size 1.27 1.27)
+				)
+				(hide yes)
+			)
+		)
 		(pin "1"
 		)
@@
 			)
 		)
+		(property "MPN" "C1523"
+			(at 173.99 44.45 0)
+			(effects
+				(font
+					(size 1.27 1.27)
+				)
+				(hide yes)
+			)
+		)
 		(pin "2"
 		)
@@
 			(at 80.01 148.59 0)
 			(effects
+				(font
+					(size 1.27 1.27)
+				)
+				(hide yes)
+			)
+		)
+		(property "MPN" "C19702"
+			(at 80.01 148.59 0)
+			(effects
