File: dac.kicad_sch (KiCad schematic)
At the start: 0 parts

Commit message: Lesson 7: ADC, DAC, and frontends
Parts:
- added C501: 10u, symbol Device:C_Small
- added C502, C505: 100n, symbol Device:C_Small
- added C503: 1u, symbol Device:C_Small
- added C504, C506: 1n, symbol Device:C_Small
- added C507: 150p, symbol Device:C_Small
- added D501: PESD3V3L1BA,115, Diode_SMD:D_SOD-323, symbol Diode:SD05_SOD323
- added J501: DOSIN-801-0031, symbol Connector:Conn_Coaxial
- added R501: 0R, symbol Device:R_Small
- added R502: 10k, symbol Device:R_Small
- added R503: 6k8, symbol Device:R_Small
- added R504: 22k, symbol Device:R_Small
- added R505: 12k, symbol Device:R_Small
- added R506: 49R9, symbol Device:R_Small
- added U501: DAC7563TDGSR, Package_SO:VSSOP-10_3x3mm_P0.5mm, symbol MissingComponents:DAC756x
- added U502: MCP6001T-E/OT, Package_TO_SOT_SMD:SOT-23-5, symbol Amplifier_Operational:MCP6001-OT
Connections:
- new net: R503.1, U501.1 (VOUT_A)
- new net: R502.1, U501.2 (VOUT_B)
- new net: C506.1, R503.2, R504.1
- new net: C504.1, R504.2, R505.1
- new net +3.3V: C501.2, C502.2, U501.9 (AVDD)
- new net +3.3VA: C505.2, U502.5 (V+)
- new net DAC_NCLR: U501.5 (~{CLR})
- new net DAC_NLDAC: U501.4 (~{LDAC})
- new net DAC_SCLK: R501.2, U501.7 (SCLK)
- new net DAC_VREF: C503.1, U501.10 (VREFIN/VREFOUT)
- new net GND: C501.1, C502.1, C503.2, C505.1, C506.2, C507.2, D501.1 (A1), J501.2 (Ext), R502.2, U501.3 (GND), U502.2 (V-)
- new net IN: D501.2 (A2), J501.1 (In), R506.2
- new net OUT_AA_BUF_IN: C507.1, R505.2, U502.3 (+)
- new net OUT_AA_BUF_OUT: C504.2, R506.1, U502.1, U502.4 (-)
- new net SPI2_MISO: U501.8 (DIN)
- new net SPI2_NSS: U501.6 (~{SYNC})
- new net SPI2_SCK: R501.1
Other:
- note added: "3rd order Butterworth anti-aliasing (low-pass filter) fc=25kHz"
- note added: "Anti-Aliasing Filter and Output Connector (BNC)"
- note added: "C(Vref,min)=150nF"
- note added: "DAC"
- note added: "DC offset (op-amp bias) generated by DAC"
- note added: "Output voltage will be in 0V to +3.3V range!"
- note added: "Rout = 50R"
- note added: "[4] DAC & Analogue Output Circuitry"

Commit message: Lesson 8: Reannotation, running ERC for schematic
Parts:
- renumbered C504 to C501, C501 to C502, C502 to C503, C505 to C504, C506 to C505, C507 to C506, C503 to C507, R503 to R501, R504 to R502, R505 to R503, R506 to R504, R501 to R505, R502 to R506, U502 to U501, U501 to U502
Connections:
- net SPI2_MISO renamed SPI2_MOSI
Other:
- note added: "Note: the course design calls for a DAC7563SDGSR. It's been replaced it with a (seemingly identical) DAC7563TDGSR, because of supply issues"
Changed lines of the file:
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@@
+		)
+	)
+	(text "Note: the course design calls for a DAC7563SDGSR.\nIt's been replaced it with a (seemingly identical) DAC7563TDGSR, because of supply issues"
+		(exclude_from_sim no)
+		(at 34.036 108.204 0)
+		(effects
+			(font
+				(size 1.27 1.27)
+				(thickness 0.254)
+				(bold yes)
+			)
+			(justify left)
 		)
 	)
@@
 		)
 	)
-	(global_label "SPI2_MISO"
+	(global_label "SPI2_MOSI"
 		(shape input)
 		(at 46.99 73.66 180)
@@
 		(on_board yes)
 		(dnp no)
-		(property "Reference" "R501"
+		(property "Reference" "R505"
 			(at 53.34 75.692 90)
 			(effects
@@
 			(project ""
 				(path "/dc1e796d-d6ca-4eeb-b725-72531775b7cc/cf59f8c7-acda-4edc-bf31-7ffb2d25aeb8"
-					(reference "R501")
+					(reference "R505")
 					(unit 1)
 				)
@@
 		(dnp no)
 		(fields_autoplaced yes)
-		(property "Reference" "C503"
+		(property "Reference" "C507"
 			(at 109.22 88.9062 0)
 			(effects
@@
 			(project ""
 				(path "/dc1e796d-d6ca-4eeb-b725-72531775b7cc/cf59f8c7-acda-4edc-bf31-7ffb2d25aeb8"
-					(reference "C503")
+					(reference "C507")
 					(unit 1)
 				)
@@
 		(dnp no)
 		(fields_autoplaced yes)
-		(property "Reference" "U501"
+		(property "Reference" "U502"
 			(at 84.7441 66.04 0)
 			(effects
@@
 			(project ""
 				(path "/dc1e796d-d6ca-4eeb-b725-72531775b7cc/cf59f8c7-acda-4edc-bf31-7ffb2d25aeb8"
-					(reference "U501")
+					(reference "U502")
 					(unit 1)
 				)
@@
 		(on_board yes)
 		(dnp no)
-		(property "Reference" "U502"
+		(property "Reference" "U501"
 			(at 180.848 71.374 0)
 			(effects
@@
 			(project "Mixed-Signal_Demo_PCB"
 				(path "/dc1e796d-d6ca-4eeb-b725-72531775b7cc/cf59f8c7-acda-4edc-bf31-7ffb2d25aeb8"
-					(reference "U502")
+					(reference "U501")
 					(unit 1)
 				)
@@
 		(dnp no)
 		(fields_autoplaced yes)
-		(property "Reference" "R503"
+		(property "Reference" "R501"
 			(at 127 68.58 90)
 			(effects
@@
 			(project "Mixed-Signal_Demo_PCB"
 				(path "/dc1e796d-d6ca-4eeb-b725-72531775b7cc/cf59f8c7-acda-4edc-bf31-7ffb2d25aeb8"
-					(reference "R503")
+					(reference "R501")
 					(unit 1)
 				)
@@
 		(dnp no)
 		(fields_autoplaced yes)
-		(property "Reference" "#PWR0502"
+		(property "Reference" "#PWR0509"
 			(at 82.55 104.14 0)
 			(effects
@@
 			(project ""
 				(path "/dc1e796d-d6ca-4eeb-b725-72531775b7cc/cf59f8c7-acda-4edc-bf31-7ffb2d25aeb8"
-					(reference "#PWR0502")
+					(reference "#PWR0509")
 					(unit 1)
 				)
@@
 		(dnp no)
 		(fields_autoplaced yes)
-		(property "Reference" "R505"
+		(property "Reference" "R503"
 			(at 147.32 68.58 90)
 			(effects
@@
 			(project "Mixed-Signal_Demo_PCB"
 				(path "/dc1e796d-d6ca-4eeb-b725-72531775b7cc/cf59f8c7-acda-4edc-bf31-7ffb2d25aeb8"
-					(reference "R505")
+					(reference "R503")
 					(unit 1)
 				)
@@
 		(dnp no)
 		(fields_autoplaced yes)
-		(property "Reference" "#PWR0509"
+		(property "Reference" "#PWR0508"
 			(at 227.33 95.25 0)
 			(effects
@@
 			(project "Mixed-Signal_Demo_PCB"
 				(path "/dc1e796d-d6ca-4eeb-b725-72531775b7cc/cf59f8c7-acda-4edc-bf31-7ffb2d25aeb8"
-					(reference "#PWR0509")
+					(reference "#PWR0508")
 					(unit 1)
 				)
@@
 		(dnp no)
 		(fields_autoplaced yes)
-		(property "Reference" "#PWR0508"
+		(property "Reference" "#PWR0507"
 			(at 153.67 93.98 0)
 			(effects
@@
 			(project "Mixed-Signal_Demo_PCB"
 				(path "/dc1e796d-d6ca-4eeb-b725-72531775b7cc/cf59f8c7-acda-4edc-bf31-7ffb2d25aeb8"
-					(reference "#PWR0508")
+					(reference "#PWR0507")
 					(unit 1)
 				)
@@
 		(on_board yes)
 		(dnp no)
-		(property "Reference" "C504"
+		(property "Reference" "C501"
 			(at 153.924 54.102 90)
 			(effects
@@
 			(project "Mixed-Signal_Demo_PCB"
 				(path "/dc1e796d-d6ca-4eeb-b725-72531775b7cc/cf59f8c7-acda-4edc-bf31-7ffb2d25aeb8"
-					(reference "C504")
+					(reference "C501")
 					(unit 1)
 				)
@@
 		(dnp no)
 		(fields_autoplaced yes)
-		(property "Reference" "C506"
+		(property "Reference" "C505"
 			(at 134.62 78.7462 0)
 			(effects
@@
 			(project "Mixed-Signal_Demo_PCB"
 				(path "/dc1e796d-d6ca-4eeb-b725-72531775b7cc/cf59f8c7-acda-4edc-bf31-7ffb2d25aeb8"
-					(reference "C506")
+					(reference "C505")
 					(unit 1)
 				)
@@
 		(dnp no)
 		(fields_autoplaced yes)
-		(property "Reference" "#PWR0507"
+		(property "Reference" "#PWR0506"
 			(at 173.99 92.71 0)
 			(effects
@@
 			(project "Mixed-Signal_Demo_PCB"
 				(path "/dc1e796d-d6ca-4eeb-b725-72531775b7cc/cf59f8c7-acda-4edc-bf31-7ffb2d25aeb8"
-					(reference "#PWR0507")
+					(reference "#PWR0506")
 					(unit 1)
 				)
@@
 		(dnp no)
 		(fields_autoplaced yes)
-		(property "Reference" "#PWR0505"
+		(property "Reference" "#PWR0504"
 			(at 162.56 73.66 0)
 			(effects
@@
 			(project "Mixed-Signal_Demo_PCB"
 				(path "/dc1e796d-d6ca-4eeb-b725-72531775b7cc/cf59f8c7-acda-4edc-bf31-7ffb2d25aeb8"
-					(reference "#PWR0505")
+					(reference "#PWR0504")
 					(unit 1)
 				)
@@
 		(dnp no)
 		(fields_autoplaced yes)
-		(property "Reference" "#PWR0504"
+		(property "Reference" "#PWR0502"
 			(at 173.99 68.58 0)
 			(effects
@@
 			(project "Mixed-Signal_Demo_PCB"
 				(path "/dc1e796d-d6ca-4eeb-b725-72531775b7cc/cf59f8c7-acda-4edc-bf31-7ffb2d25aeb8"
-					(reference "#PWR0504")
+					(reference "#PWR0502")
 					(unit 1)
 				)
@@
 		(dnp no)
 		(fields_autoplaced yes)
-		(property "Reference" "C502"
+		(property "Reference" "C503"
 			(at 73.66 59.6835 0)
 			(effects
@@
 			(project "Mixed-Signal_Demo_PCB"
 				(path "/dc1e796d-d6ca-4eeb-b725-72531775b7cc/cf59f8c7-acda-4edc-bf31-7ffb2d25aeb8"
-					(reference "C502")
+					(reference "C503")
 					(unit 1)
 				)
@@
 		(dnp no)
 		(fields_autoplaced yes)
-		(property "Reference" "R502"
+		(property "Reference" "R506"
 			(at 121.92 88.8999 0)
 			(effects
@@
 			(project ""
 				(path "/dc1e796d-d6ca-4eeb-b725-72531775b7cc/cf59f8c7-acda-4edc-bf31-7ffb2d25aeb8"
-					(reference "R502")
+					(reference "R506")
 					(unit 1)
 				)
@@
 		(dnp no)
 		(fields_autoplaced yes)
-		(property "Reference" "R506"
+		(property "Reference" "R504"
 			(at 203.2 71.12 90)
 			(effects
@@
 			(project ""
 				(path "/dc1e796d-d6ca-4eeb-b725-72531775b7cc/cf59f8c7-acda-4edc-bf31-7ffb2d25aeb8"
-					(reference "R506")
+					(reference "R504")
 					(unit 1)
 				)
@@
 		(dnp no)
 		(fields_autoplaced yes)
-		(property "Reference" "C501"
+		(property "Reference" "C502"
 			(at 63.5 59.6835 0)
 			(effects
@@
 			(project ""
 				(path "/dc1e796d-d6ca-4eeb-b725-72531775b7cc/cf59f8c7-acda-4edc-bf31-7ffb2d25aeb8"
-					(reference "C501")
+					(reference "C502")
 					(unit 1)
 				)
@@
 		(on_board yes)
 		(dnp no)
-		(property "Reference" "C505"
+		(property "Reference" "C504"
 			(at 167.64 63.246 90)
 			(effects
@@
 			(project "Mixed-Signal_Demo_PCB"
 				(path "/dc1e796d-d6ca-4eeb-b725-72531775b7cc/cf59f8c7-acda-4edc-bf31-7ffb2d25aeb8"
-					(reference "C505")
+					(reference "C504")
 					(unit 1)
 				)
@@
 		(dnp no)
 		(fields_autoplaced yes)
-		(property "Reference" "R504"
+		(property "Reference" "R502"
 			(at 137.16 68.58 90)
 			(effects
@@
 			(project "Mixed-Signal_Demo_PCB"
 				(path "/dc1e796d-d6ca-4eeb-b725-72531775b7cc/cf59f8c7-acda-4edc-bf31-7ffb2d25aeb8"
-					(reference "R504")
+					(reference "R502")
 					(unit 1)
 				)
@@
 		(dnp no)
 		(fields_autoplaced yes)
-		(property "Reference" "#PWR0506"
+		(property "Reference" "#PWR0505"
 			(at 132.08 92.71 0)
 			(effects
@@
 			(project "Mixed-Signal_Demo_PCB"
 				(path "/dc1e796d-d6ca-4eeb-b725-72531775b7cc/cf59f8c7-acda-4edc-bf31-7ffb2d25aeb8"
-					(reference "#PWR0506")
+					(reference "#PWR0505")
 					(unit 1)
 				)
@@
 		(dnp no)
 		(fields_autoplaced yes)
-		(property "Reference" "C507"
+		(property "Reference" "C506"
 			(at 156.21 78.7462 0)
 			(effects
@@
 			(project "Mixed-Signal_Demo_PCB"
 				(path "/dc1e796d-d6ca-4eeb-b725-72531775b7cc/cf59f8c7-acda-4edc-bf31-7ffb2d25aeb8"
-					(reference "C507")
-					(unit 1)
-				)
+					(reference "C506")
+					(unit 1)
+				)

Commit message: Lesson 8: Assigned most footprints. Added missing ones
Parts:
- C501, C502, C503, C504, C505, C506, C507: footprint (none) -> Capacitor_SMD:C_0402_1005Metric
- R501: footprint (none) -> Resistor_SMD:R_0603_1608Metric
- R502, R503, R504, R505, R506: footprint (none) -> Resistor_SMD:R_0402_1005Metric
Changed lines of the file:
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@@
 			)
 		)
-		(property "Footprint" ""
+		(property "Footprint" "Resistor_SMD:R_0402_1005Metric"
 			(at 53.34 77.47 0)
 			(effects
@@
 			)
 		)
-		(property "Footprint" ""
+		(property "Footprint" "Capacitor_SMD:C_0402_1005Metric"
 			(at 106.68 90.17 0)
 			(effects
@@
 			)
 		)
-		(property "Footprint" ""
+		(property "Footprint" "Resistor_SMD:R_0603_1608Metric"
 			(at 127 73.66 0)
 			(effects
@@
 			)
 		)
-		(property "Footprint" ""
+		(property "Footprint" "Resistor_SMD:R_0402_1005Metric"
 			(at 147.32 73.66 0)
 			(effects
@@
 			)
 		)
-		(property "Footprint" ""
+		(property "Footprint" "Capacitor_SMD:C_0402_1005Metric"
 			(at 153.67 57.15 0)
 			(effects
@@
 			)
 		)
-		(property "Footprint" ""
+		(property "Footprint" "Capacitor_SMD:C_0402_1005Metric"
 			(at 132.08 80.01 0)
 			(effects
@@
 			)
 		)
-		(property "Footprint" ""
+		(property "Footprint" "Capacitor_SMD:C_0402_1005Metric"
 			(at 71.12 60.96 0)
 			(effects
@@
 			)
 		)
-		(property "Footprint" ""
+		(property "Footprint" "Resistor_SMD:R_0402_1005Metric"
 			(at 119.38 90.17 0)
 			(effects
@@
 			)
 		)
-		(property "Footprint" ""
+		(property "Footprint" "Resistor_SMD:R_0402_1005Metric"
 			(at 203.2 76.2 0)
 			(effects
@@
 			)
 		)
-		(property "Footprint" ""
+		(property "Footprint" "Capacitor_SMD:C_0402_1005Metric"
 			(at 60.96 60.96 0)
 			(effects
@@
 			)
 		)
-		(property "Footprint" ""
+		(property "Footprint" "Capacitor_SMD:C_0402_1005Metric"
 			(at 167.64 66.04 0)
 			(effects
@@
 			)
 		)
-		(property "Footprint" ""
+		(property "Footprint" "Resistor_SMD:R_0402_1005Metric"
 			(at 137.16 73.66 0)
 			(effects
@@
 			)
 		)
-		(property "Footprint" ""
+		(property "Footprint" "Capacitor_SMD:C_0402_1005Metric"
 			(at 153.67 80.01 0)
 			(effects

Commit message: Lesson 11: Adjusted capacitor footprints and set up PCB defaults
Parts:
- C502, C507: footprint Capacitor_SMD:C_0402_1005Metric -> Capacitor_SMD:C_0603_1608Metric
- J501: footprint (none) -> Connector_Coaxial:BNC_Amphenol_B6252HB-NPP3G-50_Horizontal
Changed lines of the file:
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@@
 			)
 		)
-		(property "Footprint" "Capacitor_SMD:C_0402_1005Metric"
+		(property "Footprint" "Capacitor_SMD:C_0603_1608Metric"
 			(at 106.68 90.17 0)
 			(effects
@@
 			)
 		)
-		(property "Footprint" ""
+		(property "Footprint" "Connector_Coaxial:BNC_Amphenol_B6252HB-NPP3G-50_Horizontal"
 			(at 227.33 76.2 0)
 			(effects
@@
 			)
 		)
-		(property "Footprint" "Capacitor_SMD:C_0402_1005Metric"
+		(property "Footprint" "Capacitor_SMD:C_0603_1608Metric"
 			(at 60.96 60.96 0)
 			(effects

Commit message: Lesson 12: ADC and DAC
Parts:
- R501: footprint Resistor_SMD:R_0603_1608Metric -> Resistor_SMD:R_0402_1005Metric
Connections:
- net DAC_OUT_A: now reaches R501.1, U502.1 (VOUT_A)
- net DAC_OUT_B: now reaches R506.1, U502.2 (VOUT_B)
Changed lines of the file:
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@@
+		)
+	)
+	(label "DAC_OUT_B"
+		(at 104.14 77.47 0)
+		(fields_autoplaced yes)
+		(effects
+			(font
+				(size 1.27 1.27)
+			)
+			(justify left bottom)
 		)
 	)
 	(label "OUT_AA_BUF_OUT"
 		(at 177.8 91.44 0)
+		(fields_autoplaced yes)
+		(effects
+			(font
+				(size 1.27 1.27)
+			)
+			(justify left bottom)
+		)
+	)
+	(label "DAC_OUT_A"
+		(at 104.14 73.66 0)
 		(fields_autoplaced yes)
 		(effects
@@
 			)
 		)
-		(property "Footprint" "Resistor_SMD:R_0603_1608Metric"
+		(property "Footprint" "Resistor_SMD:R_0402_1005Metric"
 			(at 127 73.66 0)
 			(effects

Commit message: Assembly files
Parts:
- C501, C505: MPN (none) -> C1523
- C502: MPN (none) -> C19702
- C503, C504: MPN (none) -> C1525
- C506: MPN (none) -> C106998
- C507: MPN (none) -> C15849
- R501: footprint Resistor_SMD:R_0402_1005Metric -> Resistor_SMD:R_0603_1608Metric; MPN (none) -> C23212
- R502: MPN (none) -> C25768
- R503: MPN (none) -> C25752
- R504: MPN (none) -> C25120
- R505: MPN (none) -> C17168
- R506: MPN (none) -> C25744
Changed lines of the file:
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@@
+			)
+		)
+		(property "MPN" "C17168"
+			(at 53.34 77.47 0)
+			(effects
+				(font
+					(size 1.27 1.27)
+				)
+				(hide yes)
 			)
 		)
@@
 			)
 		)
+		(property "MPN" "C15849"
+			(at 106.68 90.17 0)
+			(effects
+				(font
+					(size 1.27 1.27)
+				)
+				(hide yes)
+			)
+		)
 		(pin "1"
 		)
@@
 			)
 		)
-		(property "Footprint" "Resistor_SMD:R_0402_1005Metric"
+		(property "Footprint" "Resistor_SMD:R_0603_1608Metric"
 			(at 127 73.66 0)
 			(effects
@@
 			)
 		)
+		(property "MPN" "C23212"
+			(at 127 73.66 0)
+			(effects
+				(font
+					(size 1.27 1.27)
+				)
+				(hide yes)
+			)
+		)
 		(pin "1"
 		)
@@
 		)
 		(property "Description" "Resistor, small symbol"
+			(at 147.32 73.66 0)
+			(effects
+				(font
+					(size 1.27 1.27)
+				)
+				(hide yes)
+			)
+		)
+		(property "MPN" "C25752"
 			(at 147.32 73.66 0)
 			(effects
@@
 			)
 		)
+		(property "MPN" "C1523"
+			(at 153.67 57.15 0)
+			(effects
+				(font
+					(size 1.27 1.27)
+				)
+				(hide yes)
+			)
+		)
 		(pin "2"
 		)
@@
 			)
 		)
+		(property "MPN" "C1523"
+			(at 132.08 80.01 0)
+			(effects
+				(font
+					(size 1.27 1.27)
+				)
+				(hide yes)
+			)
+		)
 		(pin "2"
 		)
@@
 			)
 		)
+		(property "MPN" "C1525"
+			(at 71.12 60.96 0)
+			(effects
+				(font
+					(size 1.27 1.27)
+				)
+				(hide yes)
+			)
+		)
 		(pin "1"
 		)
@@
 			)
 		)
+		(property "MPN" "C25744"
+			(at 119.38 90.17 0)
+			(effects
+				(font
+					(size 1.27 1.27)
+				)
+				(hide yes)
+			)
+		)
 		(pin "1"
 		)
@@
 			)
 		)
+		(property "MPN" "C25120"
+			(at 203.2 76.2 0)
+			(effects
+				(font
+					(size 1.27 1.27)
+				)
+				(hide yes)
+			)
+		)
 		(pin "2"
 		)
@@
 			)
 		)
+		(property "MPN" "C19702"
+			(at 60.96 60.96 0)
+			(effects
+				(font
+					(size 1.27 1.27)
+				)
+				(hide yes)
+			)
+		)
 		(pin "1"
 		)
@@
 		)
 		(property "Description" "Unpolarized capacitor, small symbol"
+			(at 167.64 66.04 0)
+			(effects
+				(font
+					(size 1.27 1.27)
+				)
+				(hide yes)
+			)
+		)
+		(property "MPN" "C1525"
 			(at 167.64 66.04 0)
 			(effects
@@
 			)
 		)
+		(property "MPN" "C25768"
+			(at 137.16 73.66 0)
+			(effects
+				(font
+					(size 1.27 1.27)
+				)
+				(hide yes)
+			)
+		)
 		(pin "1"
 		)
@@
 			(at 153.67 80.01 0)
 			(effects
+				(font
+					(size 1.27 1.27)
+				)
+				(hide yes)
+			)
+		)
+		(property "MPN" "C106998"
+			(at 153.67 80.01 0)
+			(effects
