File: mcu.kicad_sch (KiCad schematic)
At the start: 0 parts

Commit message: Lesson 6: MCU and USB module
Parts:
- added C301: 10u, symbol Device:C_Small
- added C302, C303, C304, C305, C311, C312, C313: 100n, symbol Device:C_Small
- added C306: 10n, symbol Device:C_Small
- added C307, C308: 1u, symbol Device:C_Small
- added C309, C310: 10p, symbol Device:C_Small
- added D301: LED_RGB_E6C1206RGBC3UDA, symbol Device:LED_RGBA
- added D302, D303, D304, D305, D306: PESD3V3L1BA,115, Diode_SMD:D_SOD-323, symbol Diode:SD05_SOD323
- added FL301: CMF3216F-900-2P-T, symbol Device:Filter_EMI_LL_1423
- added J301: USB_C_Receptacle_USB2.0_16P, symbol Connector:USB_C_Receptacle_USB2.0_16P
- added J302: 2x5x1.27mm, symbol Connector_Generic:Conn_02x05_Odd_Even
- added L301: 10n, symbol Device:L_Small
- added R301, R302, R307: 10k, symbol Device:R_Small
- added R303, R304: 5k1, symbol Device:R_Small
- added R305: 0R, symbol Device:R_Small
- added R306: 1k5, symbol Device:R_Small
- added R308, R309, R310: 1k, symbol Device:R_Small
- added R311, R312, R313, R314: 49R9, symbol Device:R_Small
- added U301: STM32F103CBTx, Package_QFP:LQFP-48_7x7mm_P0.5mm, symbol MCU_ST_STM32F1:STM32F103CBTx
- added U302: USBLC6-2SC6, Package_TO_SOT_SMD:SOT-23-6, symbol Power_Protection:USBLC6-2SC6
- added Y301: 16MHz, symbol Device:Crystal_GND24
Connections:
- new net: D303.2 (A2), J302.2 (Pin_2), R311.1
- new net: D305.2 (A2), J302.6 (Pin_6), R313.1
- new net: D304.2 (A2), J302.4 (Pin_4), R312.1
- new net: J301.A5 (CC1), R303.1
- new net: D306.2 (A2), J302.10 (Pin_10), R314.1
- new net: J301.B5 (CC2), R304.1
- new net +3.3V: C301.1, C302.1, C303.1, C304.1, C305.1, C308.1, C311.1, D301.4 (A), D302.2 (A2), J302.1 (Pin_1), L301.2, R302.1, R306.1, R307.1, U301.1 (VBAT), U301.24 (VDD), U301.36 (VDD), U301.48 (VDD)
- new net +3.3VA: C306.1, C307.1, L301.1, U301.9 (VDDA)
- new net BOOT0: R301.2, U301.44 (BOOT0)
- new net DAC_NCLR: U301.21 (PB10)
- new net DAC_NLDAC: U301.22 (PB11)
- new net GND: C301.2, C302.2, C303.2, C304.2, C305.2, C306.2, C307.2, C308.2, C309.2, C310.2, C311.2, C312.1, C313.2, D302.1 (A1), D303.1 (A1), D304.1 (A1), D305.1 (A1), D306.1 (A1), J301.A1 (GND), J301.A12 (GND), J301.B1 (GND), J301.B12 (GND), J302.3 (Pin_3), J302.5 (Pin_5), J302.9 (Pin_9), R301.1, R303.2, R304.2, U301.23 (VSS), U301.35 (VSS), U301.47 (VSS), U301.8 (VSSA), U302.2 (GND), Y301.2, Y301.4
- new net HSE_IN: C309.1, U301.5 (PD0), Y301.1
- new net HSE_OUT: R305.2, U301.6 (PD1)
- new net LED_B_k: D301.3 (BK), R310.2
- new net LED_G_k: D301.2 (GK), R309.2
- new net LED_R_k: D301.1 (RK), R308.2
- new net NRST: C313.1, R314.2, U301.7 (NRST)
- new net SPI1_MISO: U301.16 (PA6)
- new net SPI1_NSS: R302.2, U301.14 (PA4)
- new net SPI1_SCK: U301.15 (PA5)
- new net SPI2_MOSI: U301.28 (PB15)
- new net SPI2_NSS: R307.2, U301.25 (PB12)
- new net SPI2_SCK: U301.26 (PB13)
- new net SWCLK: R312.2, U301.37 (PA14)
- new net SWDIO: R311.2, U301.34 (PA13)
- new net SWO: R313.2, U301.39 (PB3)
- new net TIM4_CH1: R308.1, U301.42 (PB6)
- new net TIM4_CH2: R309.1, U301.43 (PB7)
- new net TIM4_CH3: R310.1, U301.45 (PB8)
- new net USB_CMC_D+: U302.4 (I/O2)
- new net USB_CMC_D-: FL301.1, U302.6 (I/O1)
- new net USB_CONN_D+: J301.A6 (D+), J301.B6 (D+), U302.3 (I/O2)
- new net USB_CONN_D-: J301.A7 (D-), J301.B7 (D-), U302.1 (I/O1)
- new net USB_D+: FL301.3, R306.2, U301.33 (PA12)
- new net USB_D-: FL301.4, U301.32 (PA11)
- new net VBUS: C312.2, J301.A4 (VBUS), J301.A9 (VBUS), J301.B4 (VBUS), J301.B9 (VBUS), U302.5 (VBUS)
- new net XTAL_IN: C310.1, R305.1, Y301.3
- no-connect marks 0 -> 24
Other:
- note added: "CL=10pF ESR=80R"
- note added: "Common-Mode Chocke Impedance: 90R"
- note added: "Crystall app note: AN2867"
- note added: "MCU (STM32F1)"
- note added: "RGB LED"
- note added: "SWD Header"
- note added: "Signal Path: Connector <-> ESD Protection <-> Common-Mode Choke <-> Pull-Up <-> MCU"
- note added: "USB Type C"
- note added: "USB app note: AN4879"
- note added: "[2] Microcontroller & USB"

Commit message: Lesson 8: Reannotation, running ERC for schematic
Parts:
- renumbered C312 to C311, C311 to C312, R311 to R309, R309 to R310, R312 to R311, R313 to R312, R310 to R313
Connections:
- net USB_CMC_D+: now also FL301.2
Changed lines of the file:
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@@
 	)
 	(junction
+		(at 220.98 49.53)
+		(diameter 0)
+		(color 0 0 0 0)
+	)
+	(junction
 		(at 121.92 44.45)
 		(diameter 0)
@@
 	(wire
 		(pts
-			(xy 186.69 121.92) (xy 210.82 121.92)
+			(xy 186.69 123.19) (xy 210.82 123.19)
 		)
 		(stroke
@@
 	(wire
 		(pts
+			(xy 220.98 49.53) (xy 220.98 48.26)
+		)
+		(stroke
+			(width 0)
+			(type default)
+		)
+	)
+	(wire
+		(pts
 			(xy 81.28 111.76) (xy 83.82 111.76)
 		)
@@
 	(wire
 		(pts
-			(xy 220.98 52.07) (xy 220.98 48.26)
+			(xy 220.98 52.07) (xy 220.98 49.53)
 		)
 		(stroke
@@
 	)
 	(label "USB_CMC_D+"
-		(at 186.69 121.92 0)
+		(at 186.69 123.19 0)
 		(fields_autoplaced yes)
 		(effects
@@
 		(on_board yes)
 		(dnp no)
-		(property "Reference" "R311"
+		(property "Reference" "R309"
 			(at 143.51 160.02 90)
 			(effects
@@
 			(project ""
 				(path "/dc1e796d-d6ca-4eeb-b725-72531775b7cc/60576906-eb66-49e0-a3d8-17c57ae5d0d1"
-					(reference "R311")
+					(reference "R309")
 					(unit 1)
 				)
@@
 		(dnp no)
 		(fields_autoplaced yes)
-		(property "Reference" "#PWR0321"
+		(property "Reference" "#PWR0319"
 			(at 90.17 162.56 0)
 			(effects
@@
 			(project "Mixed-Signal_Demo_PCB"
 				(path "/dc1e796d-d6ca-4eeb-b725-72531775b7cc/60576906-eb66-49e0-a3d8-17c57ae5d0d1"
-					(reference "#PWR0321")
+					(reference "#PWR0319")
 					(unit 1)
 				)
@@
 		(on_board yes)
 		(dnp no)
-		(property "Reference" "R310"
+		(property "Reference" "R313"
 			(at 39.37 167.132 90)
 			(effects
@@
 			(project "Mixed-Signal_Demo_PCB"
 				(path "/dc1e796d-d6ca-4eeb-b725-72531775b7cc/60576906-eb66-49e0-a3d8-17c57ae5d0d1"
-					(reference "R310")
+					(reference "R313")
 					(unit 1)
 				)
@@
 	)
 	(symbol
+		(lib_id "power:PWR_FLAG")
+		(at 220.98 49.53 90)
+		(unit 1)
+		(exclude_from_sim no)
+		(in_bom yes)
+		(on_board yes)
+		(dnp no)
+		(fields_autoplaced yes)
+		(property "Reference" "#FLG0301"
+			(at 219.075 49.53 0)
+			(effects
+				(font
+					(size 1.27 1.27)
+				)
+				(hide yes)
+			)
+		)
+		(property "Value" "PWR_FLAG"
+			(at 217.17 49.5299 90)
+			(effects
+				(font
+					(size 1.27 1.27)
+				)
+				(justify left)
+			)
+		)
+		(property "Footprint" ""
+			(at 220.98 49.53 0)
+			(effects
+				(font
+					(size 1.27 1.27)
+				)
+				(hide yes)
+			)
+		)
+		(property "Datasheet" "~"
+			(at 220.98 49.53 0)
+			(effects
+				(font
+					(size 1.27 1.27)
+				)
+				(hide yes)
+			)
+		)
+		(property "Description" "Special symbol for telling ERC where power comes from"
+			(at 220.98 49.53 0)
+			(effects
+				(font
+					(size 1.27 1.27)
+				)
+				(hide yes)
+			)
+		)
+		(pin "1"
+		)
+		(instances
+			(project ""
+				(path "/dc1e796d-d6ca-4eeb-b725-72531775b7cc/60576906-eb66-49e0-a3d8-17c57ae5d0d1"
+					(reference "#FLG0301")
+					(unit 1)
+				)
+			)
+		)
+	)
+	(symbol
 		(lib_id "Device:C_Small")
 		(at 62.23 48.26 0)
@@
 		(dnp no)
 		(fields_autoplaced yes)
-		(property "Reference" "#PWR0314"
+		(property "Reference" "#PWR0318"
 			(at 99.06 139.7 0)
 			(effects
@@
 			(project "Mixed-Signal_Demo_PCB"
 				(path "/dc1e796d-d6ca-4eeb-b725-72531775b7cc/60576906-eb66-49e0-a3d8-17c57ae5d0d1"
-					(reference "#PWR0314")
+					(reference "#PWR0318")
 					(unit 1)
 				)
@@
 		(dnp no)
 		(fields_autoplaced yes)
-		(property "Reference" "#PWR0307"
+		(property "Reference" "#PWR0304"
 			(at 220.98 52.07 0)
 			(effects
@@
 			(project ""
 				(path "/dc1e796d-d6ca-4eeb-b725-72531775b7cc/60576906-eb66-49e0-a3d8-17c57ae5d0d1"
-					(reference "#PWR0307")
+					(reference "#PWR0304")
 					(unit 1)
 				)
@@
 		(dnp no)
 		(fields_autoplaced yes)
-		(property "Reference" "C312"
+		(property "Reference" "C311"
 			(at 193.0463 83.82 90)
 			(effects
@@
 			(project ""
 				(path "/dc1e796d-d6ca-4eeb-b725-72531775b7cc/60576906-eb66-49e0-a3d8-17c57ae5d0d1"
-					(reference "C312")
+					(reference "C311")
 					(unit 1)
 				)
@@
 		(dnp no)
 		(fields_autoplaced yes)
-		(property "Reference" "#PWR0305"
+		(property "Reference" "#PWR0306"
 			(at 132.08 58.42 0)
 			(effects
@@
 			(project "Mixed-Signal_Demo_PCB"
 				(path "/dc1e796d-d6ca-4eeb-b725-72531775b7cc/60576906-eb66-49e0-a3d8-17c57ae5d0d1"
-					(reference "#PWR0305")
+					(reference "#PWR0306")
 					(unit 1)
 				)
@@
 		(dnp no)
 		(fields_autoplaced yes)
-		(property "Reference" "C311"
+		(property "Reference" "C312"
 			(at 68.58 166.3762 0)
 			(effects
@@
 			(project ""
 				(path "/dc1e796d-d6ca-4eeb-b725-72531775b7cc/60576906-eb66-49e0-a3d8-17c57ae5d0d1"
-					(reference "C311")
+					(reference "C312")
 					(unit 1)
 				)
@@
 		(dnp no)
 		(fields_autoplaced yes)
-		(property "Reference" "#PWR0313"
+		(property "Reference" "#PWR0316"
 			(at 60.96 110.49 0)
 			(effects
@@
 			(project "Mixed-Signal_Demo_PCB"
 				(path "/dc1e796d-d6ca-4eeb-b725-72531775b7cc/60576906-eb66-49e0-a3d8-17c57ae5d0d1"
-					(reference "#PWR0313")
+					(reference "#PWR0316")
 					(unit 1)
 				)
@@
 		(dnp no)
 		(fields_autoplaced yes)
-		(property "Reference" "#PWR0306"
+		(property "Reference" "#PWR0307"
 			(at 153.67 58.42 0)
 			(effects
@@
 			(project "Mixed-Signal_Demo_PCB"
 				(path "/dc1e796d-d6ca-4eeb-b725-72531775b7cc/60576906-eb66-49e0-a3d8-17c57ae5d0d1"
-					(reference "#PWR0306")
+					(reference "#PWR0307")
 					(unit 1)
 				)
@@
 		(dnp no)
 		(fields_autoplaced yes)
-		(property "Reference" "#PWR0311"
+		(property "Reference" "#PWR0314"
 			(at 35.56 99.06 0)
 			(effects
@@
 			(project "Mixed-Signal_Demo_PCB"
 				(path "/dc1e796d-d6ca-4eeb-b725-72531775b7cc/60576906-eb66-49e0-a3d8-17c57ae5d0d1"
-					(reference "#PWR0311")
+					(reference "#PWR0314")
 					(unit 1)
 				)
@@
 		(dnp no)
 		(fields_autoplaced yes)
-		(property "Reference" "#PWR0319"
+		(property "Reference" "#PWR0313"
 			(at 187.96 97.79 0)
 			(effects
@@
 			(project "Mixed-Signal_Demo_PCB"
 				(path "/dc1e796d-d6ca-4eeb-b725-72531775b7cc/60576906-eb66-49e0-a3d8-17c57ae5d0d1"
-					(reference "#PWR0319")
+					(reference "#PWR0313")
 					(unit 1)
 				)
@@
 		(dnp no)
 		(fields_autoplaced yes)
-		(property "Reference" "#PWR0315"
+		(property "Reference" "#PWR0320"
 			(at 66.04 166.37 0)
 			(effects
@@
 			(project ""
 				(path "/dc1e796d-d6ca-4eeb-b725-72531775b7cc/60576906-eb66-49e0-a3d8-17c57ae5d0d1"
-					(reference "#PWR0315")
+					(reference "#PWR0320")
 					(unit 1)
 				)
@@
 		(dnp no)
 		(fields_autoplaced yes)
-		(property "Reference" "#PWR0320"
+		(property "Reference" "#PWR0310"
 			(at 191.77 74.93 0)
 			(effects
@@
 			(project "Mixed-Signal_Demo_PCB"
 				(path "/dc1e796d-d6ca-4eeb-b725-72531775b7cc/60576906-eb66-49e0-a3d8-17c57ae5d0d1"
-					(reference "#PWR0320")
+					(reference "#PWR0310")
 					(unit 1)
 				)
@@
 		(dnp no)
 		(fields_autoplaced yes)
-		(property "Reference" "#PWR0318"
+		(property "Reference" "#PWR0317"
 			(at 201.93 115.57 0)
 			(effects
@@
 			(project "Mixed-Signal_Demo_PCB"
 				(path "/dc1e796d-d6ca-4eeb-b725-72531775b7cc/60576906-eb66-49e0-a3d8-17c57ae5d0d1"
-					(reference "#PWR0318")
+					(reference "#PWR0317")
 					(unit 1)
 				)
@@
 		(dnp no)
 		(fields_autoplaced yes)
-		(property "Reference" "#PWR0312"
+		(property "Reference" "#PWR0315"
 			(at 240.03 99.06 0)
 			(effects
@@
 			(project ""
 				(path "/dc1e796d-d6ca-4eeb-b725-72531775b7cc/60576906-eb66-49e0-a3d8-17c57ae5d0d1"
-					(reference "#PWR0312")
+					(reference "#PWR0315")
 					(unit 1)
 				)
@@
 		(on_board yes)
 		(dnp no)
-		(property "Reference" "R313"
+		(property "Reference" "R312"
 			(at 143.51 165.1 90)
 			(effects
@@
 			(project "Mixed-Signal_Demo_PCB"
 				(path "/dc1e796d-d6ca-4eeb-b725-72531775b7cc/60576906-eb66-49e0-a3d8-17c57ae5d0d1"
-					(reference "R313")
+					(reference "R312")
 					(unit 1)
 				)
@@
 		(on_board yes)
 		(dnp no)
-		(property "Reference" "R312"
+		(property "Reference" "R311"
 			(at 143.51 162.56 90)
 			(effects
@@
 			(project "Mixed-Signal_Demo_PCB"
 				(path "/dc1e796d-d6ca-4eeb-b725-72531775b7cc/60576906-eb66-49e0-a3d8-17c57ae5d0d1"
-					(reference "R312")
+					(reference "R311")
 					(unit 1)
 				)
@@
 		(on_board yes)
 		(dnp no)
-		(property "Reference" "R309"
+		(property "Reference" "R310"
 			(at 39.37 162.052 90)
 			(effects
@@
 			(project "Mixed-Signal_Demo_PCB"
 				(path "/dc1e796d-d6ca-4eeb-b725-72531775b7cc/60576906-eb66-49e0-a3d8-17c57ae5d0d1"
-					(reference "R309")
+					(reference "R310")
 					(unit 1)
 				)
@@
 		(dnp no)
 		(fields_autoplaced yes)
-		(property "Reference" "#PWR0317"
+		(property "Reference" "#PWR0312"
 			(at 201.93 91.44 0)
 			(effects
@@
 			(project "Mixed-Signal_Demo_PCB"
 				(path "/dc1e796d-d6ca-4eeb-b725-72531775b7cc/60576906-eb66-49e0-a3d8-17c57ae5d0d1"
-					(reference "#PWR0317")
+					(reference "#PWR0312")
 					(unit 1)
 				)
@@
 		(dnp no)
 		(fields_autoplaced yes)
-		(property "Reference" "#PWR0304"
+		(property "Reference" "#PWR0305"
 			(at 40.64 58.42 0)
 			(effects
@@
 			(project ""
 				(path "/dc1e796d-d6ca-4eeb-b725-72531775b7cc/60576906-eb66-49e0-a3d8-17c57ae5d0d1"
-					(reference "#PWR0304")
+					(reference "#PWR0305")
 					(unit 1)
 				)
@@
 		(dnp no)
 		(fields_autoplaced yes)
-		(property "Reference" "#PWR0310"
+		(property "Reference" "#PWR0311"
 			(at 147.32 85.09 0)
 			(effects
@@
 			(project "Mixed-Signal_Demo_PCB"
 				(path "/dc1e796d-d6ca-4eeb-b725-72531775b7cc/60576906-eb66-49e0-a3d8-17c57ae5d0d1"
-					(reference "#PWR0310")
+					(reference "#PWR0311")
 					(unit 1)
 				)
@@
 		(on_board yes)
 		(dnp no)
-		(property "Reference" "#PWR0316"
+		(property "Reference" "#PWR0321"
 			(at 66.04 177.8 0)
 			(effects
@@
 			(project ""
 				(path "/dc1e796d-d6ca-4eeb-b725-72531775b7cc/60576906-eb66-49e0-a3d8-17c57ae5d0d1"
-					(reference "#PWR0316")
+					(reference "#PWR0321")
 					(unit 1)
 				)

Commit message: Lesson 8: Assigned most footprints. Added missing ones
Parts:
- C301, C302, C303, C304, C305, C306, C307, C308, C309, C310, C311, C312, C313: footprint (none) -> Capacitor_SMD:C_0402_1005Metric
- D301: footprint (none) -> Missing_Footprints:E6C1206RGBC3UDA; symbol Device:LED_RGBA -> Device:LED_GARB
- FL301: footprint (none) -> Missing_Footprints:CMF3216F; MPN (none) -> C963740
- L301: footprint (none) -> Inductor_SMD:L_0402_1005Metric
- R301, R302, R303, R304, R305, R306, R307, R308, R309, R310, R311, R312, R313, R314: footprint (none) -> Resistor_SMD:R_0402_1005Metric
Connections:
- net +3.3V: now also D301.2 (A); no longer D301.4 (A)
- net LED_B_k: now also D301.4 (BK); no longer D301.3 (BK)
- net LED_G_k: now also D301.1 (GK); no longer D301.2 (GK)
- net LED_R_k: now also D301.3 (RK); no longer D301.1 (RK)
Other:
- note added: "Crystal app note: AN2867"
- note removed: "Crystall app note: AN2867"
Changed lines of the file:
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@@
 	)
 	(junction
-		(at 220.98 49.53)
-		(diameter 0)
-		(color 0 0 0 0)
-	)
-	(junction
 		(at 121.92 44.45)
 		(diameter 0)
@@
 	(wire
 		(pts
+			(xy 240.03 90.17) (xy 240.03 92.71)
+		)
+		(stroke
+			(width 0)
+			(type default)
+		)
+	)
+	(wire
+		(pts
 			(xy 134.62 166.37) (xy 146.05 166.37)
 		)
@@
 	(wire
 		(pts
-			(xy 220.98 49.53) (xy 220.98 48.26)
+			(xy 220.98 48.26) (xy 220.98 52.07)
 		)
 		(stroke
@@
 	(wire
 		(pts
-			(xy 240.03 90.17) (xy 240.03 92.71)
-		)
-		(stroke
-			(width 0)
-			(type default)
-		)
-	)
-	(wire
-		(pts
 			(xy 207.01 101.6) (xy 220.98 101.6)
 		)
@@
 	(wire
 		(pts
-			(xy 220.98 52.07) (xy 220.98 49.53)
-		)
-		(stroke
-			(width 0)
-			(type default)
-		)
-	)
-	(wire
-		(pts
 			(xy 127 163.83) (xy 146.05 163.83)
 		)
@@
 		)
 	)
-	(text "Crystall app note: AN2867"
+	(text "Crystal app note: AN2867"
 		(exclude_from_sim no)
 		(at 39.116 64.77 0)
@@
 			)
 		)
-		(property "Footprint" ""
+		(property "Footprint" "Resistor_SMD:R_0402_1005Metric"
 			(at 148.59 161.29 0)
 			(effects
@@
 			)
 		)
-		(property "Footprint" ""
+		(property "Footprint" "Missing_Footprints:CMF3216F"
 			(at 215.9 114.3 0)
 			(effects
@@
 			)
 		)
+		(property "MPN" "C963740"
+			(at 215.9 120.65 0)
+			(effects
+				(font
+					(size 1.27 1.27)
+				)
+				(hide yes)
+			)
+		)
 		(pin "4"
 		)
@@
 	)
 	(symbol
-		(lib_id "Device:LED_RGBA")
+		(lib_id "Device:LED_GARB")
 		(at 55.88 163.83 0)
 		(unit 1)
@@
 			)
 		)
-		(property "Footprint" ""
+		(property "Footprint" "Missing_Footprints:E6C1206RGBC3UDA"
 			(at 55.88 165.1 0)
 			(effects
@@
 			)
 		)
-		(property "Description" "RGB LED, red/green/blue/anode"
+		(property "Description" "RGB LED, green/anode/red/blue"
 			(at 55.88 163.83 0)
 			(effects
@@
 			)
 		)
-		(property "Footprint" ""
+		(property "Footprint" "Resistor_SMD:R_0402_1005Metric"
 			(at 41.91 168.91 0)
 			(effects
@@
 			)
 		)
-		(property "Footprint" ""
+		(property "Footprint" "Capacitor_SMD:C_0402_1005Metric"
 			(at 154.94 177.8 0)
 			(effects
@@
 	)
 	(symbol
-		(lib_id "power:PWR_FLAG")
-		(at 220.98 49.53 90)
-		(unit 1)
-		(exclude_from_sim no)
-		(in_bom yes)
-		(on_board yes)
-		(dnp no)
-		(fields_autoplaced yes)
-		(property "Reference" "#FLG0301"
-			(at 219.075 49.53 0)
-			(effects
-				(font
-					(size 1.27 1.27)
-				)
-				(hide yes)
-			)
-		)
-		(property "Value" "PWR_FLAG"
-			(at 217.17 49.5299 90)
-			(effects
-				(font
-					(size 1.27 1.27)
-				)
-				(justify left)
-			)
-		)
-		(property "Footprint" ""
-			(at 220.98 49.53 0)
-			(effects
-				(font
-					(size 1.27 1.27)
-				)
-				(hide yes)
-			)
-		)
-		(property "Datasheet" "~"
-			(at 220.98 49.53 0)
-			(effects
-				(font
-					(size 1.27 1.27)
-				)
-				(hide yes)
-			)
-		)
-		(property "Description" "Special symbol for telling ERC where power comes from"
-			(at 220.98 49.53 0)
-			(effects
-				(font
-					(size 1.27 1.27)
-				)
-				(hide yes)
-			)
-		)
-		(pin "1"
-		)
-		(instances
-			(project ""
-				(path "/dc1e796d-d6ca-4eeb-b725-72531775b7cc/60576906-eb66-49e0-a3d8-17c57ae5d0d1"
-					(reference "#FLG0301")
-					(unit 1)
-				)
-			)
-		)
-	)
-	(symbol
 		(lib_id "Device:C_Small")
 		(at 62.23 48.26 0)
@@
 			)
 		)
-		(property "Footprint" ""
+		(property "Footprint" "Capacitor_SMD:C_0402_1005Metric"
 			(at 62.23 48.26 0)
 			(effects
@@
 			)
 		)
-		(property "Footprint" ""
+		(property "Footprint" "Capacitor_SMD:C_0402_1005Metric"
 			(at 193.04 90.17 0)
 			(effects
@@
 			)
 		)
-		(property "Footprint" ""
+		(property "Footprint" "Resistor_SMD:R_0402_1005Metric"
 			(at 191.77 63.5 0)
 			(effects
@@
 			)
 		)
-		(property "Footprint" ""
+		(property "Footprint" "Resistor_SMD:R_0402_1005Metric"
 			(at 148.59 171.45 0)
 			(effects
@@
 			)
 		)
-		(property "Footprint" ""
+		(property "Footprint" "Capacitor_SMD:C_0402_1005Metric"
 			(at 60.96 86.36 0)
 			(effects
@@
 			)
 		)
-		(property "Footprint" ""
+		(property "Footprint" "Capacitor_SMD:C_0402_1005Metric"
 			(at 66.04 167.64 0)
 			(effects
@@
 			)
 		)
-		(property "Footprint" ""
+		(property "Footprint" "Capacitor_SMD:C_0402_1005Metric"
 			(at 35.56 86.36 0)
 			(effects
@@
 			)
 		)
-		(property "Footprint" ""
+		(property "Footprint" "Resistor_SMD:R_0402_1005Metric"
 			(at 68.58 71.12 0)
 			(effects
@@
 			)
 		)
-		(property "Footprint" ""
+		(property "Footprint" "Capacitor_SMD:C_0402_1005Metric"
 			(at 132.08 48.26 0)
 			(effects
@@
 			)
 		)
-		(property "Footprint" ""
+		(property "Footprint" "Inductor_SMD:L_0402_1005Metric"
 			(at 142.24 44.45 0)
 			(effects
@@
 			)
 		)
-		(property "Footprint" ""
+		(property "Footprint" "Capacitor_SMD:C_0402_1005Metric"
 			(at 82.55 48.26 0)
 			(effects
@@
 			)
 		)
-		(property "Footprint" ""
+		(property "Footprint" "Resistor_SMD:R_0402_1005Metric"
 			(at 200.66 63.5 0)
 			(effects
@@
 			)
 		)
-		(property "Footprint" ""
+		(property "Footprint" "Resistor_SMD:R_0402_1005Metric"
 			(at 147.32 83.82 0)
 			(effects
@@
 			)
 		)
-		(property "Footprint" ""
+		(property "Footprint" "Resistor_SMD:R_0402_1005Metric"
 			(at 68.58 63.5 0)
 			(effects
@@
 			)
 		)
-		(property "Footprint" ""
+		(property "Footprint" "Capacitor_SMD:C_0402_1005Metric"
 			(at 121.92 48.26 0)
 			(effects
@@
 			)
 		)
-		(property "Footprint" ""
+		(property "Footprint" "Resistor_SMD:R_0402_1005Metric"
 			(at 41.91 158.75 0)
 			(effects
@@
 			)
 		)
-		(property "Footprint" ""
+		(property "Footprint" "Resistor_SMD:R_0402_1005Metric"
 			(at 148.59 166.37 0)
 			(effects
@@
 			)
 		)
-		(property "Footprint" ""
+		(property "Footprint" "Capacitor_SMD:C_0402_1005Metric"
 			(at 52.07 48.26 0)
 			(effects
@@
 			)
 		)
-		(property "Footprint" ""
+		(property "Footprint" "Resistor_SMD:R_0402_1005Metric"
 			(at 128.27 63.5 0)
 			(effects
@@
 			)
 		)
-		(property "Footprint" ""
+		(property "Footprint" "Resistor_SMD:R_0402_1005Metric"
 			(at 148.59 163.83 0)
 			(effects
@@
 			)
 		)
-		(property "Footprint" ""
+		(property "Footprint" "Capacitor_SMD:C_0402_1005Metric"
 			(at 40.64 48.26 0)
 			(effects
@@
 			)
 		)
-		(property "Footprint" ""
+		(property "Footprint" "Resistor_SMD:R_0402_1005Metric"
 			(at 41.91 163.83 0)
 			(effects
@@
 			)
 		)
-		(property "Footprint" ""
+		(property "Footprint" "Capacitor_SMD:C_0402_1005Metric"
 			(at 153.67 48.26 0)
 			(effects
@@
 			)
 		)
-		(property "Footprint" ""
+		(property "Footprint" "Resistor_SMD:R_0402_1005Metric"
 			(at 60.96 110.49 0)
 			(effects
@@
 			)
 		)
-		(property "Footprint" ""
+		(property "Footprint" "Capacitor_SMD:C_0402_1005Metric"
 			(at 72.39 48.26 0)
 			(effects

Commit message: Lesson 11: Adjusted capacitor footprints and set up PCB defaults
Parts:
- C301, C307, C308: footprint Capacitor_SMD:C_0402_1005Metric -> Capacitor_SMD:C_0603_1608Metric
- J301: footprint (none) -> Connector_USB:USB_C_Receptacle_G-Switch_GT-USB-7010ASV
- J302: footprint (none) -> Connector_PinHeader_1.27mm:PinHeader_2x05_P1.27mm_Vertical_SMD
- Y301: footprint (none) -> Crystal:Crystal_SMD_3225-4Pin_3.2x2.5mm
Changed lines of the file:
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@@
 			)
 		)
-		(property "Footprint" ""
+		(property "Footprint" "Crystal:Crystal_SMD_3225-4Pin_3.2x2.5mm"
 			(at 48.26 78.74 0)
 			(effects
@@
 			)
 		)
-		(property "Footprint" "Capacitor_SMD:C_0402_1005Metric"
+		(property "Footprint" "Capacitor_SMD:C_0603_1608Metric"
 			(at 132.08 48.26 0)
 			(effects
@@
 			)
 		)
-		(property "Footprint" ""
+		(property "Footprint" "Connector_USB:USB_C_Receptacle_G-Switch_GT-USB-7010ASV"
 			(at 236.22 67.31 0)
 			(effects
@@
 			)
 		)
-		(property "Footprint" "Capacitor_SMD:C_0402_1005Metric"
+		(property "Footprint" "Capacitor_SMD:C_0603_1608Metric"
 			(at 40.64 48.26 0)
 			(effects
@@
 			)
 		)
-		(property "Footprint" "Capacitor_SMD:C_0402_1005Metric"
+		(property "Footprint" "Capacitor_SMD:C_0603_1608Metric"
 			(at 153.67 48.26 0)
 			(effects
@@
 			)
 		)
-		(property "Footprint" ""
+		(property "Footprint" "Connector_PinHeader_1.27mm:PinHeader_2x05_P1.27mm_Vertical_SMD"
 			(at 106.68 166.37 0)
 			(effects
